File: emg_headband/hardware/emg_afe/kicad/emg_wearable_revA.kicad_sch (KiCad schematic)
At the start: 60 parts, among them J1 ELECTRODES (TRS), J2 ISO UART (DNP), J3 LiPo, U1 INA333AIDGKR, U2 XIAO ESP32-S3, U3 OPA2333AIDR, U4 OPA2333AIDR, U5 ISO7721DWVR (DNP)

Commit message: EMG Rev A: automatic USB/battery power path and LP5907 analog LDO
Replace the ferrite off the XIAO 3V3 with a passive power path (Schottky
from USB 5V, AO3401A from the battery) into an LP5907 3.0 V low-noise
LDO enabled by the XIAO 3V3. Analog rail renamed +3V0_A, VMID now 1.5 V.
ERC clean.

Co-Authored-By: Claude Opus 5.5 (1M context) <noreply@anthropic.com>
Parts:
- removed FB1: 600R@100MHz, Inductor_SMD:L_0603_1608Metric, symbol Device:FerriteBead_Small
- added C107: 10uF, Capacitor_SMD:C_0603_1608Metric, symbol Device:C
- added D101: B5819W, Diode_SMD:D_SOD-123, symbol Device:D_Schottky
- added Q101: AO3401A, Package_TO_SOT_SMD:SOT-23, symbol Transistor_FET:AO3401A
- added R104: 100k, Resistor_SMD:R_0603_1608Metric, symbol Device:R
- added U6: LP5907MFX-3.0, Package_TO_SOT_SMD:SOT-23-5, symbol Regulator_Linear:LP5907MFX-3.0
- C101: value 10uF -> 1uF; LCSC C19702 -> C15849
- TP1: value +3V3_A -> +3V0_A
Connections:
- net +3V3: now also U6.3 (EN)
- net AGND: now also C107.2, R104.2, U6.2 (GND)
- net VBAT: now also Q101.3 (D)
- net VBUS: now reaches U2.14 (5V)
- net VBUS: now also D101.2 (A), Q101.1 (G), R104.1
- net +3V3_A renamed +3V0_A
- net +3V0_A: now also U6.5 (OUT)
- new net VSYS: C107.1, D101.1 (K), Q101.2 (S), U6.1 (IN)
Other:
- note added: "POWER: USB 5V / LiPo auto power path -> LP5907 3.0 V low-noise LDO -> +3V0_A (EN from XIAO 3V3)"
- note added: "SAFETY: with electrodes on the body and USB-C plugged in, run the laptop on battery, unplugged from mains, or use a simulated input instead of electrodes. Keep the isolation gap under U5 free of copper."
- note added: "VMID = 1.5 V: divider, U3A buffer, 47R + 1uF. INA REF from VMID_BUF"
- note removed: "POWER: XIAO 3V3 -> FB1 -> +3V3_A (AFE only live when ESP32 is powered)"
- note removed: "SAFETY: with electrodes on the body and USB-C plugged in, run the laptop on battery, unplugged from mains, or use a simulated input instead of electrodes. No charging while worn. Keep the isolation gap under U5 free of copper."
- note removed: "VMID = 1.65 V: divider, U3A buffer, 47R + 1uF. INA REF from VMID_BUF"

Commit message: EMG Rev A: TRS jack per channel and flip-lock FPC for flex arrays
Add CH2/CH3 TRS jacks (J4, J5) and a 12-pin Hirose FH12 FPC (J6) wired
in parallel with all three jacks, with AGND guards between channels.
CH2/CH3 are not yet wired to a front end. ERC clean.

Co-Authored-By: Claude Opus 5.5 (1M context) <noreply@anthropic.com>
Parts:
- added J4: CH2 ELECTRODES (TRS), Connector_Audio:Jack_3.5mm_CUI_SJ-3523-SMT_Horizontal, symbol Connector_Audio:AudioJack3
- added J5: CH3 ELECTRODES (TRS), Connector_Audio:Jack_3.5mm_CUI_SJ-3523-SMT_Horizontal, symbol Connector_Audio:AudioJack3
- added J6: FLEX ARRAY (FPC 12P 0.5mm), Connector_FFC-FPC:Hirose_FH12-12S-0.5SH_1x12-1MP_P0.50mm_Horizontal, symbol Connector_Generic_MountingPin:Conn_01x12_MountingPin
Connections:
- net AGND: now also J6.1 (Pin_1), J6.5 (Pin_5), J6.9 (Pin_9), J6.MP (MountPin)
- net ELEC_N: now also J6.3 (Pin_3)
- net ELEC_P: now also J6.2 (Pin_2)
- net ELEC_REF: now also J6.4 (Pin_4)
- new net ELEC2_N: J4.R, J6.7 (Pin_7)
- new net ELEC2_P: J4.T, J6.6 (Pin_6)
- new net ELEC2_REF: J4.S, J6.8 (Pin_8)
- new net ELEC3_N: J5.R, J6.11 (Pin_11)
- new net ELEC3_P: J5.T, J6.10 (Pin_10)
- new net ELEC3_REF: J5.S, J6.12 (Pin_12)
Other:
- note added: "ELECTRODES: J1/J4/J5 TRS per channel (T +, R -, S REF). J6 = 2 mm flip-lock FPC for a future flex array, in parallel with the TRS jacks: use one or the other. J6 1/5/9 + MP = AGND guards. CH2/CH3 join the front end once the ADC choice is made."
- note added: "INA333 G1 = 6"
- note added: "POWER: USB/LiPo auto path -> LP5907 3.0 V LDO -> +3V0_A"
- note removed: "INA333 G1 = 1 + 100k/20k = 6"
- note removed: "POWER: USB 5V / LiPo auto power path -> LP5907 3.0 V low-noise LDO -> +3V0_A (EN from XIAO 3V3)"

Commit message: EMG Rev A: replace discrete chain with ADS1298, 1 to 3 channels
Three TRS jacks and the FPC feed an ADS1298 through 22k/1nF input RC,
with all REF sleeves on one RLD net (330k series, datasheet 1M||1.5nF
feedback). SPI, DRDY, START, RESET to the XIAO; internal clock and
reference; unused inputs tied to AVDD per datasheet. Power path and
debug sections carried over. README rewritten with the reviewed
requirements. ERC: 0 errors, 2 datasheet-expected warnings.

Co-Authored-By: Claude Opus 5.5 (1M context) <noreply@anthropic.com>
Parts:
- removed C103, C104, C302: 1uF, Capacitor_SMD:C_0603_1608Metric, symbol Device:C
- removed C105, C106, C301: 100nF, Capacitor_SMD:C_0603_1608Metric, symbol Device:C
- removed C401: 10nF C0G, Capacitor_SMD:C_0603_1608Metric, symbol Device:C
- removed C501, C502: 15nF C0G, Capacitor_SMD:C_0603_1608Metric, symbol Device:C
- removed C601: 2.2nF C0G, Capacitor_SMD:C_0603_1608Metric, symbol Device:C
- removed C602: 1.8nF C0G, Capacitor_SMD:C_0603_1608Metric, symbol Device:C
- removed C603: 6.8nF C0G, Capacitor_SMD:C_0603_1608Metric, symbol Device:C
- removed C604: 1nF C0G, Capacitor_SMD:C_0603_1608Metric, symbol Device:C
- removed D201, D202: BAV199 (DNP), Package_TO_SOT_SMD:SOT-23, symbol Device:D_Dual_Series_AKC
- removed JP401: GAIN (1-2: x66, 2-3: x240), Jumper:SolderJumper-3_P1.3mm_Bridged12_RoundedPad1.0x1.5mm_NumberLabels, symbol Jumper:SolderJumper_3_Bridged12
- removed R301: 20k, Resistor_SMD:R_0603_1608Metric, symbol Device:R
- removed R401: 820k, Resistor_SMD:R_0603_1608Metric, symbol Device:R
- removed R402: 10k, Resistor_SMD:R_0603_1608Metric, symbol Device:R
- removed R403: 100k, Resistor_SMD:R_0603_1608Metric, symbol Device:R
- removed R404: 390k, Resistor_SMD:R_0603_1608Metric, symbol Device:R
- removed R501, R502: 1k, Resistor_SMD:R_0603_1608Metric, symbol Device:R
- removed R601, R602: 165k, Resistor_SMD:R_0603_1608Metric, symbol Device:R
- removed R603, R604: 127k, Resistor_SMD:R_0603_1608Metric, symbol Device:R
- removed TP9: AGND, TestPoint:TestPoint_Pad_D1.0mm, symbol Connector:TestPoint
- removed U1: INA333AIDGKR, Package_SO:VSSOP-8_3x3mm_P0.65mm, symbol Amplifier_Instrumentation:INA333xxDGK
- removed U3, U4: OPA2333AIDR, Package_SO:SOIC-8_3.9x4.9mm_P1.27mm, symbol Amplifier_Operational:OPA2333xxD
- added C111: 1.5nF C0G, Capacitor_SMD:C_0603_1608Metric, symbol Device:C
- added C112, C118: 10uF, Capacitor_SMD:C_0603_1608Metric, symbol Device:C
- added C113, C119, C120, C122: 100nF, Capacitor_SMD:C_0603_1608Metric, symbol Device:C
- added C114: 22uF, Capacitor_SMD:C_0603_1608Metric, symbol Device:C
- added C115, C116, C117, C121: 1uF, Capacitor_SMD:C_0603_1608Metric, symbol Device:C
- added C204, C205, C206: 1nF C0G, Capacitor_SMD:C_0603_1608Metric, symbol Device:C
- added R105, R106: 10k, Resistor_SMD:R_0603_1608Metric, symbol Device:R
- added R206: 22k, Resistor_SMD:R_0603_1608Metric, symbol Device:R
- added U1: ADS1298IPAGR, Package_QFP:TQFP-64_10x10mm_P0.5mm, symbol Analog_ADC:ADS1298xPAG
- C201, C202: value 22pF C0G -> 1nF C0G; LCSC C1653 -> C163508
- C203: value 220pF C0G -> 1nF C0G; LCSC C27675 -> C163508
- J1: value ELECTRODES (TRS) -> CH1 (TRS)
- J3: value LiPo -> LiPo (protected)
- J4: value CH2 ELECTRODES (TRS) -> CH2 (TRS)
- J5: value CH3 ELECTRODES (TRS) -> CH3 (TRS)
- R101: value 100k -> 1M; LCSC C25803 -> C22935
- R102: value 100k -> 330k; LCSC C25803 -> C23137
- R103: value 47R -> 10k; LCSC C23182 -> C25804
- R201, R202, R205: value 100k -> 22k; LCSC C25803 -> C31850
- R203, R204: value 10M -> 22k; LCSC C7250 -> C31850
- TP2: value VMID -> +3V3
- TP4: value INA_OUT -> VSYS
- TP5: value GAIN_OUT -> RLD_OUT
- TP6: value AAF_MID -> ADS_DRDY
- TP7: value AAF_OUT -> SPI_SCK
- TP8: value ADC_OUT -> AGND
Connections:
- net AAF_MID is gone; now on net ADS_DRDY: TP6.1
- net AAF_OUT is gone; now on net SPI_SCK: TP7.1
- net ELEC3_REF is gone; now on net RLD_ELEC: J5.S, J6.12 (Pin_12)
- net INA_OUT is gone; now on net VSYS: TP4.1
- net VMID_BUF is gone; now on net +3V3: R103.1
- net VMID_RAW is gone; now on net RLD_OUT: R101.2, R102.1
- net +3V0_A: now also C118.1, C119.1, C120.1, U1.1 (IN8N), U1.10 (IN4P), U1.17 (TESTP_PACE_OUT1), U1.18 (TESTP_PACE_OUT2), U1.19 (AVDD), U1.2 (IN8P), U1.21 (AVDD), U1.22 (AVDD), U1.3 (IN7N), U1.4 (IN7P), U1.5 (IN6N), U1.54 (AVDD1), U1.56 (AVDD), U1.59 (AVDD), U1.6 (IN6P), U1.7 (IN5N), U1.8 (IN5P), U1.9 (IN4N); no longer R101.1
- net +3V3: now also TP2.1, C121.1, C122.1, R105.1, R106.1, U1.48 (DVDD), U1.50 (DVDD), U1.52 (CLKSEL)
- net AGND: now also C203.2, TP8.1, C112.2, C113.2, C114.2, C115.2, C116.2, C117.2, C118.2, C119.2, C120.2, C121.2, C122.2, C204.2, C205.2, C206.2, U1.20 (AVSS), U1.23 (AVSS), U1.25 (VREFN), U1.31 (RESV1), U1.32 (AVSS), U1.33 (DGND), U1.41 (DAISY_IN), U1.49 (DGND), U1.51 (DGND), U1.53 (AVSS1), U1.57 (AVSS), U1.58 (AVSS); no longer R102.2
- net ELEC2_N: now also R204.1
- net ELEC2_P: now also R203.1
- net ELEC3_N: now also R206.1
- net ELEC3_P: now also R205.1
- net SPI_MISO: now reaches U2.10 (D9_IO8)
- net SPI_MISO: now also U1.43 (DOUT)
- net SPI_MOSI: now reaches U2.11 (D10_IO9)
- net SPI_MOSI: now also U1.34 (DIN)
- net ADS_CS: now reaches U2.4 (D3_IO4)
- net ADS_CS: now also R103.2, U1.39 (~{CS})
- net ADS_DRDY: now reaches U2.5 (D4_IO5)
- net ADS_DRDY: now also U1.47 (~{DRDY})
- net SPI_SCK: now reaches U2.9 (D8_IO7)
- net SPI_SCK: now also U1.40 (SCLK)
- net ADC_OUT renamed ADS_RESET
- net ADS_RESET: now also R105.2, U1.36 (~{RESET}); no longer TP8.1
- net ELEC2_REF renamed RLD_ELEC
- net RLD_ELEC: now also J1.S, J6.4 (Pin_4), R102.2, U1.62 (RLDIN)
- net ELEC_N renamed ELEC1_N
- net ELEC_P renamed ELEC1_P
- removed net ELEC_REF: J1.S, J6.4 (Pin_4), R205.1
- net GAIN_OUT renamed RLD_OUT
- net RLD_OUT: now also C111.2, U1.63 (RLDOUT)
- net IN_N renamed CH1_N
- net CH1_N: now also U1.15 (IN1N); no longer C203.2, R204.1
- net IN_P renamed CH1_P
- net CH1_P: now also U1.16 (IN1P); no longer C203.1, R203.1
- removed net VMID: R103.2, R203.2, R204.2, R205.2, TP2.1
- net VMID_MON renamed ADS_START
- net ADS_START: now also U1.38 (START)
- new net ADS_PWDN: R106.2, U1.35 (~{PWDN})
- new net CH2_N: C204.1, R204.2, U1.13 (IN2N)
- new net CH2_P: C203.1, R203.2, U1.14 (IN2P)
- new net CH3_N: C206.1, R206.2, U1.11 (IN3N)
- new net CH3_P: C205.1, R205.2, U1.12 (IN3P)
- new net RLD_INV: C111.1, R101.1, U1.61 (RLDINV)
- new net VCAP1: C114.1, U1.28 (VCAP1)
- new net VCAP2: C115.1, U1.30 (VCAP2)
- new net VCAP3: C116.1, U1.55 (VCAP3)
- new net VCAP4: C117.1, U1.26 (VCAP4)
- new net VREFP: C112.1, C113.1, U1.24 (VREFP)
- no-connect marks 8 -> 12
Other:
- note added: "ADS1298: CH1-CH3 used, CH4-CH8 and TESTP tied to AVDD per datasheet (power down in firmware). 1, 2 or 3 channels by mode, no rework. HPF/LPF in firmware: capture ~0.5 Hz up at 4 kSPS+. Lead-off detection and RLD channel selection are firmware settings. Internal clock (CLKSEL high), internal 2.4 V reference."
- note added: "ELECTRODES: one TRS per channel (T +, R -, S REF). All sleeves share RLD_ELEC, so use 3 REF electrodes (9 total) or one (7 total). J6 FPC is in parallel with the jacks: use one or the other. J6 1/5/9 + MP = AGND guards."
- note added: "INPUT RC: 22k series (limits fault and plug-insertion current) + 1nF C0G to AGND, ~7 kHz. ADS1298 oversamples at 512 kHz, so this is the only anti-alias filter needed."
- note added: "LiPo: J3 wires to the XIAO underside BAT+/BAT- pads (U2 pins 15/16). XIAO is hand-soldered."
- note added: "POWER: USB 5V (D101) / LiPo (Q101) auto power path -> VSYS -> U6 LP5907 3.0 V -> +3V0_A (ADS1298 AVDD) U6 EN = XIAO 3V3, so the AFE is off whenever the ESP32 is off. DVDD = XIAO 3V3."
- note added: "RLD: 1M || 1.5nF feedback, 330k series to the REF electrode(s) limits DC fault current to <10 uA."
- note added: "SAFETY: with electrodes on the body and USB-C plugged in, run the laptop on battery, unplugged from mains, or use a simulated input. Charge while worn only from an isolated (Class II) charger. Keep the isolation gap under U5 free of copper. LAYOUT: keep U1 and its supply away from the XIAO antenna."
- note removed: "ADC: 1k + 15nF C0G (10.6 kHz) into D0. VMID_MON into D1, subtract in firmware"
- note removed: "ANTI-ALIAS: 4th-order Butterworth Sallen-Key, fc ~480 Hz. R x10, C /10 vs README so all caps are 0603 C0G"
- note removed: "ELECTRODE INPUT: 100k series, 10M bias to VMID, RFI filter. D201/D202 clamps DNP"
- note removed: "ELECTRODES: J1/J4/J5 TRS per channel (T +, R -, S REF). J6 = 2 mm flip-lock FPC for a future flex array, in parallel with the TRS jacks: use one or the other. J6 1/5/9 + MP = AGND guards. CH2/CH3 join the front end once the ADC choice is made."
- note removed: "HPF 19.4 Hz, U3B gain: JP401 1-2 = 100k (G2 11, total 66), 2-3 = 390k (G2 40, total 240)"
- note removed: "INA333 G1 = 6"
- note removed: "LiPo: J3 wires to the XIAO underside BAT+/BAT- pads (U2 pins 15/16). XIAO is hand-soldered, not JLC assembled."
- note removed: "POWER: USB/LiPo auto path -> LP5907 3.0 V LDO -> +3V0_A"
- note removed: "SAFETY: with electrodes on the body and USB-C plugged in, run the laptop on battery, unplugged from mains, or use a simulated input instead of electrodes. Keep the isolation gap under U5 free of copper."
- note removed: "Stage A Q 0.55 fc 485 Hz | Stage B Q 1.30 fc 480 Hz"
- note removed: "VMID = 1.5 V: divider, U3A buffer, 47R + 1uF. INA REF from VMID_BUF"

Commit message: EMG Rev A: 1 mm Hirose FH34SRJ FPC for the flex array
Custom footprint drawn from the Hirose land pattern; J6 now C424659.

Co-Authored-By: Claude Opus 5.5 (1M context) <noreply@anthropic.com>
Parts:
- J6: value FLEX ARRAY (FPC 12P 0.5mm) -> FLEX ARRAY (FPC 12P 0.5mm, 1mm tall); footprint Connector_FFC-FPC:Hirose_FH12-12S-0.5SH_1x12-1MP_P0.50mm_Horizontal -> emg_wearable:Hirose_FH34SRJ-12S-0.5SH_1x12-1MP_P0.50mm_Horizontal; LCSC C88360 -> C424659; MPN Hirose FH12-12S-0.5SH(55) -> Hirose FH34SRJ-12S-0.5SH(50)
Changed lines of the file:
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@@
 			)
 		)
-		(property "Value" "FLEX ARRAY (FPC 12P 0.5mm)"
+		(property "Value" "FLEX ARRAY (FPC 12P 0.5mm, 1mm tall)"
 			(at 30.48 212.09 0)
 			(show_name no)
@@
 			)
 		)
-		(property "Footprint" "Connector_FFC-FPC:Hirose_FH12-12S-0.5SH_1x12-1MP_P0.50mm_Horizontal"
+		(property "Footprint" "emg_wearable:Hirose_FH34SRJ-12S-0.5SH_1x12-1MP_P0.50mm_Horizontal"
 			(at 30.48 228.6 0)
 			(hide yes)
@@
 			)
 		)
-    (property "LCSC" "C88360" (at 30.48 228.6 0)
+    (property "LCSC" "C424659" (at 30.48 228.6 0)
       (effects (font (size 1.27 1.27)) (hide yes))
     )
-    (property "MPN" "Hirose FH12-12S-0.5SH(55)" (at 30.48 228.6 0)
+    (property "MPN" "Hirose FH34SRJ-12S-0.5SH(50)" (at 30.48 228.6 0)
       (effects (font (size 1.27 1.27)) (hide yes))
     )

Commit message: EMG Rev A: fit 2.5x1in flex board, start layout
One 3.5 mm jack (CH1) plus the 1 mm FPC for CH1-CH3, isolated UART
dropped, LiPo on solder pads, XIAO soldered by its castellations.
Board outline 63.5 x 25.4 mm with flex design rules and first-pass
placement (XIAO left with USB-C down, ADS1298 middle, jack/FPC right).
Not routed yet.

Co-Authored-By: Claude Opus 5.5 (1M context) <noreply@anthropic.com>
Parts:
- removed C701, C702: 100nF (DNP), Capacitor_SMD:C_0603_1608Metric, symbol Device:C
- removed J2: ISO UART (DNP), Connector_PinHeader_2.54mm:PinHeader_1x04_P2.54mm_Vertical, symbol Connector:Conn_01x04_Pin
- removed J4: CH2 (TRS), Connector_Audio:Jack_3.5mm_CUI_SJ-3523-SMT_Horizontal, symbol Connector_Audio:AudioJack3
- removed J5: CH3 (TRS), Connector_Audio:Jack_3.5mm_CUI_SJ-3523-SMT_Horizontal, symbol Connector_Audio:AudioJack3
- removed U5: ISO7721DWVR (DNP), Package_SO:SOIC-8_7.5x5.85mm_P1.27mm, symbol Isolator:ISO7721DWV
- J3: value LiPo (protected) -> LiPo pads (protected cell); footprint Connector_JST:JST_PH_S2B-PH-K_1x02_P2.00mm_Horizontal -> emg_wearable:LiPo_SolderPads_2x2.0x3.0mm_P3.5mm; LCSC C173752 -> (none); MPN JST S2B-PH-K-S -> (none)
- J6: value FLEX ARRAY (FPC 12P 0.5mm, 1mm tall) -> FLEX ARRAY CH1-3 (FPC 12P 0.5mm, 1mm tall)
- U2: footprint emg_wearable:XIAO_ESP32S3_THT -> emg_wearable:XIAO_ESP32S3_SMD
Connections:
- net UART_RX: no longer names the net of U2.8 (RX_IO44)
- net UART_TX: no longer names the net of U2.7 (TX_IO43)
- no-connect marks 12 -> 14
Other:
- note added: "ELECTRODES: J1 TRS for CH1 (T +, R -, S REF). J6 1 mm FPC carries CH1-CH3 for a flex array or breakout, in parallel with J1 for CH1: use one or the other. All REF pins share RLD_ELEC. J6 1/5/9 + MP = AGND guards."
- note added: "LiPo: J3 = two solder pads for the protected LiPo leads. XIAO BAT+/BAT- (U2 15/16) are under the module."
- note added: "SAFETY: with electrodes on the body and USB-C plugged in, run the laptop on battery, unplugged from mains, or use a simulated input. Charge while worn only from an isolated (Class II) charger. LAYOUT: keep U1 and its supply away from the XIAO antenna."
- note removed: "DEBUG: USB serial over the XIAO USB-C is the default. U5/J2 isolated UART is optional and DNP. Populate U5, C701, C702, J2 if needed; J2 side is powered by the USB-UART adapter (3.3 or 5 V)."
- note removed: "ELECTRODES: one TRS per channel (T +, R -, S REF). All sleeves share RLD_ELEC, so use 3 REF electrodes (9 total) or one (7 total). J6 FPC is in parallel with the jacks: use one or the other. J6 1/5/9 + MP = AGND guards."
- note removed: "LiPo: J3 wires to the XIAO underside BAT+/BAT- pads (U2 pins 15/16). XIAO is hand-soldered."
- note removed: "SAFETY: with electrodes on the body and USB-C plugged in, run the laptop on battery, unplugged from mains, or use a simulated input. Charge while worn only from an isolated (Class II) charger. Keep the isolation gap under U5 free of copper. LAYOUT: keep U1 and its supply away from the XIAO antenna."

Commit message: EMG Rev A: route the 2.5x1in flex board and add JLC fab outputs
Freerouting pass plus fixes: FPC pins reordered to match the input RC
column, input filters spaced out, SPI clock moved to XIAO D5, SCLK/DRDY
test points dropped, top-layer keepout under the XIAO. AGND pours on
both layers with stitching vias, silkscreen refs hidden, back-side
labels, stiffener areas on User.1. DRC clean except J1 silk at the
board edge. Gerbers, drill, JLC BOM and CPL in kicad/fab/.

Co-Authored-By: Claude Opus 5.5 (1M context) <noreply@anthropic.com>
Parts:
- removed TP6: ADS_DRDY, TestPoint:TestPoint_Pad_D1.0mm, symbol Connector:TestPoint
- removed TP7: SPI_SCK, TestPoint:TestPoint_Pad_D1.0mm, symbol Connector:TestPoint
Connections:
- net ELEC1_N: now also J6.10 (Pin_10); no longer J6.3 (Pin_3)
- net ELEC1_P: now also J6.11 (Pin_11); no longer J6.2 (Pin_2)
- net ELEC2_N: now also J6.6 (Pin_6); no longer J6.7 (Pin_7)
- net ELEC2_P: now also J6.7 (Pin_7); no longer J6.6 (Pin_6)
- net ELEC3_N: now also J6.2 (Pin_2); no longer J6.11 (Pin_11)
- net ELEC3_P: now also J6.3 (Pin_3); no longer J6.10 (Pin_10)
- net SPI_SCK: now also U2.6 (D5_IO6); no longer U2.9 (D8_IO7)
Changed lines of the file:
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@@
 		)
 	)
-	(label "SPI_SCK"
-		(at 68.58 66.04 0)
-		(effects
-			(font
-				(size 1.27 1.27)
-			)
-			(justify left bottom)
-		)
-	)
 	(label "SPI_MISO"
 		(at 68.58 63.5 0)
@@
 	)
 	(no_connect
-		(at 43.18000000000001 66.04)
-	)
-	(no_connect
 		(at 149.86 50.8)
 	)
@@
 		)
 	)
-	(label "ELEC1_P"
-		(at 25.4 218.44 180)
-		(effects
-			(font
-				(size 1.27 1.27)
-			)
-			(justify right bottom)
-		)
-	)
-	(label "ELEC1_N"
-		(at 25.4 220.98 180)
-		(effects
-			(font
-				(size 1.27 1.27)
-			)
-			(justify right bottom)
-		)
-	)
 	(label "RLD_ELEC"
 		(at 25.4 223.51999999999998 180)
@@
 		)
 	)
-	(label "ELEC2_P"
-		(at 25.4 228.6 180)
-		(effects
-			(font
-				(size 1.27 1.27)
-			)
-			(justify right bottom)
-		)
-	)
-	(label "ELEC2_N"
-		(at 25.4 231.14 180)
-		(effects
-			(font
-				(size 1.27 1.27)
-			)
-			(justify right bottom)
-		)
-	)
 	(label "RLD_ELEC"
 		(at 25.4 233.68 180)
@@
 		)
 	)
-	(label "ELEC3_P"
-		(at 25.4 238.76 180)
-		(effects
-			(font
-				(size 1.27 1.27)
-			)
-			(justify right bottom)
-		)
-	)
-	(label "ELEC3_N"
-		(at 25.4 241.29999999999998 180)
-		(effects
-			(font
-				(size 1.27 1.27)
-			)
-			(justify right bottom)
-		)
-	)
 	(label "RLD_ELEC"
 		(at 25.4 243.84 180)
@@
 	(symbol
 		(lib_id "Connector:TestPoint")
-		(at 330.2 50.8 0)
-		(unit 1)
-		(body_style 1)
-		(exclude_from_sim no)
-		(in_bom yes)
-		(on_board yes)
-		(in_pos_files yes)
-		(dnp no)
-		(property "Reference" "TP6"
-			(at 330.2 46.99 0)
-			(show_name no)
-			(do_not_autoplace no)
-			(effects
-				(font
-					(size 1.27 1.27)
-				)
-			)
-		)
-		(property "Value" "ADS_DRDY"
-			(at 330.2 45.72 0)
-			(show_name no)
-			(do_not_autoplace no)
-			(effects
-				(font
-					(size 1.27 1.27)
-				)
-			)
-		)
-		(property "Footprint" "TestPoint:TestPoint_Pad_D1.0mm"
-			(at 335.28 50.8 0)
-			(hide yes)
-			(show_name no)
-			(do_not_autoplace no)
-			(effects
-				(font
-					(size 1.27 1.27)
-				)
-			)
-		)
-		(property "Datasheet" ""
-			(at 335.28 50.8 0)
-			(hide yes)
-			(show_name no)
-			(do_not_autoplace no)
-			(effects
-				(font
-					(size 1.27 1.27)
-				)
-			)
-		)
-		(property "Description" "test point"
-			(at 330.2 50.8 0)
-			(hide yes)
-			(show_name no)
-			(do_not_autoplace no)
-			(effects
-				(font
-					(size 1.27 1.27)
-				)
-			)
-		)
-		(pin "1"
-		)
-		(instances
-			(project "emg_wearable_revA"
-				(path "/83f63b6a-8dba-42d8-8ff4-81f3e69fb851"
-					(reference "TP6")
-					(unit 1)
-				)
-			)
-		)
-	)
-	(symbol
-		(lib_id "Connector:TestPoint")
-		(at 342.9 50.8 0)
-		(unit 1)
-		(body_style 1)
-		(exclude_from_sim no)
-		(in_bom yes)
-		(on_board yes)
-		(in_pos_files yes)
-		(dnp no)
-		(property "Reference" "TP7"
-			(at 342.9 46.99 0)
-			(show_name no)
-			(do_not_autoplace no)
-			(effects
-				(font
-					(size 1.27 1.27)
-				)
-			)
-		)
-		(property "Value" "SPI_SCK"
-			(at 342.9 45.72 0)
-			(show_name no)
-			(do_not_autoplace no)
-			(effects
-				(font
-					(size 1.27 1.27)
-				)
-			)
-		)
-		(property "Footprint" "TestPoint:TestPoint_Pad_D1.0mm"
-			(at 347.98 50.8 0)
-			(hide yes)
-			(show_name no)
-			(do_not_autoplace no)
-			(effects
-				(font
-					(size 1.27 1.27)
-				)
-			)
-		)
-		(property "Datasheet" ""
-			(at 347.98 50.8 0)
-			(hide yes)
-			(show_name no)
-			(do_not_autoplace no)
-			(effects
-				(font
-					(size 1.27 1.27)
-				)
-			)
-		)
-		(property "Description" "test point"
-			(at 342.9 50.8 0)
-			(hide yes)
-			(show_name no)
-			(do_not_autoplace no)
-			(effects
-				(font
-					(size 1.27 1.27)
-				)
-			)
-		)
-		(pin "1"
-		)
-		(instances
-			(project "emg_wearable_revA"
-				(path "/83f63b6a-8dba-42d8-8ff4-81f3e69fb851"
-					(reference "TP7")
-					(unit 1)
-				)
-			)
-		)
-	)
-	(symbol
-		(lib_id "Connector:TestPoint")
 		(at 355.6 50.8 0)
 		(unit 1)
@@
 		)
 	)
-	(label "ADS_DRDY"
-		(at 330.2 50.8 270)
-		(effects
-			(font
-				(size 1.27 1.27)
-			)
-			(justify right bottom)
-		)
-	)
-	(label "SPI_SCK"
-		(at 342.9 50.8 270)
-		(effects
-			(font
-				(size 1.27 1.27)
-			)
-			(justify right bottom)
-		)
-	)
 	(label "AGND"
 		(at 355.6 50.8 270)
@@
 		(at 68.58 68.58)
 	)
+	(label "ELEC3_N"
+		(at 25.4 218.44 180)
+		(effects
+			(font
+				(size 1.27 1.27)
+			)
+			(justify right bottom)
+		)
+	)
+	(label "ELEC3_P"
+		(at 25.4 220.98 180)
+		(effects
+			(font
+				(size 1.27 1.27)
+			)
+			(justify right bottom)
+		)
+	)
+	(label "ELEC2_N"
+		(at 25.4 228.6 180)
+		(effects
+			(font
+				(size 1.27 1.27)
+			)
+			(justify right bottom)
+		)
+	)
+	(label "ELEC2_P"
+		(at 25.4 231.14 180)
+		(effects
+			(font
+				(size 1.27 1.27)
+			)
+			(justify right bottom)
+		)
+	)
+	(label "ELEC1_N"
+		(at 25.4 238.76 180)
+		(effects
+			(font
+				(size 1.27 1.27)
+			)
+			(justify right bottom)
+		)
+	)
+	(label "ELEC1_P"
+		(at 25.4 241.29999999999998 180)
+		(effects
+			(font
+				(size 1.27 1.27)
+			)
+			(justify right bottom)
+		)
+	)
+	(label "SPI_SCK"
+		(at 43.18000000000001 66.04 180)
+		(effects
+			(font
+				(size 1.27 1.27)
+			)
+			(justify right bottom)
+		)
+	)
+	(no_connect
+		(at 68.58 66.04)
+	)
 	(sheet_instances
