File: emg_headband/hardware/emg_afe/kicad/emg_wearable_revA.kicad_sch (KiCad schematic)
At the start: 47 parts, among them J1 CH1 (TRS), J3 LiPo pads (protected cell), J6 FLEX ARRAY CH1-3 (FPC 12P 0.5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, Q101 AO3401A, U1 ADS1298IPAGR, U2 XIAO ESP32-S3, U6 LP5907MFX-3.0

Commit message: EMG Rev A: shorten flex board to 57 mm, face the FPC outward
J6 rotated so its FPC opening (mounting-tab side) is on the board edge;
FPC pinout back to CH1 at pins 2-4. Input RC filters moved next to J6,
test pads moved to the back under the RC block. Board 57 x 25.4 mm,
re-routed, AGND pours and stitching vias, stiffener outlines updated.
DRC clean except J1 silk at the board edge. Fab outputs regenerated.

Co-Authored-By: Claude Opus 5.5 (1M context) <noreply@anthropic.com>
Connections:
- net ELEC1_N: now also J6.3 (Pin_3); no longer J6.10 (Pin_10)
- net ELEC1_P: now also J6.2 (Pin_2); no longer J6.11 (Pin_11)
- net ELEC2_N: now also J6.7 (Pin_7); no longer J6.6 (Pin_6)
- net ELEC2_P: now also J6.6 (Pin_6); no longer J6.7 (Pin_7)
- net ELEC3_N: now also J6.11 (Pin_11); no longer J6.2 (Pin_2)
- net ELEC3_P: now also J6.10 (Pin_10); no longer J6.3 (Pin_3)
Changed lines of the file:
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@@
 		(at 68.58 68.58)
-	)
-	(label "ELEC3_N"
-		(at 25.4 218.44 180)
-		(effects
-			(font
-				(size 1.27 1.27)
-			)
-			(justify right bottom)
-		)
-	)
-	(label "ELEC3_P"
-		(at 25.4 220.98 180)
-		(effects
-			(font
-				(size 1.27 1.27)
-			)
-			(justify right bottom)
-		)
-	)
-	(label "ELEC2_N"
-		(at 25.4 228.6 180)
-		(effects
-			(font
-				(size 1.27 1.27)
-			)
-			(justify right bottom)
-		)
-	)
-	(label "ELEC2_P"
-		(at 25.4 231.14 180)
-		(effects
-			(font
-				(size 1.27 1.27)
-			)
-			(justify right bottom)
-		)
-	)
-	(label "ELEC1_N"
-		(at 25.4 238.76 180)
-		(effects
-			(font
-				(size 1.27 1.27)
-			)
-			(justify right bottom)
-		)
-	)
-	(label "ELEC1_P"
-		(at 25.4 241.29999999999998 180)
-		(effects
-			(font
-				(size 1.27 1.27)
-			)
-			(justify right bottom)
-		)
 	)
 	(label "SPI_SCK"
@@
 		(at 68.58 66.04)
 	)
+	(label "ELEC1_P"
+		(at 25.4 218.44 180)
+		(effects
+			(font
+				(size 1.27 1.27)
+			)
+			(justify right bottom)
+		)
+	)
+	(label "ELEC1_N"
+		(at 25.4 220.98 180)
+		(effects
+			(font
+				(size 1.27 1.27)
+			)
+			(justify right bottom)
+		)
+	)
+	(label "ELEC2_P"
+		(at 25.4 228.6 180)
+		(effects
+			(font
+				(size 1.27 1.27)
+			)
+			(justify right bottom)
+		)
+	)
+	(label "ELEC2_N"
+		(at 25.4 231.14 180)
+		(effects
+			(font
+				(size 1.27 1.27)
+			)
+			(justify right bottom)
+		)
+	)
+	(label "ELEC3_P"
+		(at 25.4 238.76 180)
+		(effects
+			(font
+				(size 1.27 1.27)
+			)
+			(justify right bottom)
+		)
+	)
+	(label "ELEC3_N"
+		(at 25.4 241.29999999999998 180)
+		(effects
+			(font
+				(size 1.27 1.27)
+			)
+			(justify right bottom)
+		)
+	)
 	(sheet_instances

Commit message: EMG Rev A: ESP32-S3-MINI-1 on board instead of the XIAO
Replace the hand-soldered XIAO with an ESP32-S3-MINI-1-N8 (antenna at
the board end, copper kept out), HRO USB-C with CC resistors and
USBLC6 ESD, MCP73831 LiPo charger and AP2112K 3.3 V regulator on VSYS.
ADS1298 SPI on IO12-IO18; EN RC plus EN/BOOT test pads instead of
buttons. Board 62.5 x 25.4 mm, re-placed and re-routed, AGND pours,
stiffener outlines updated. ERC: 0 errors (2 datasheet-expected
warnings). DRC: clean apart from connector/module silk at the edge.
JLC BOM/CPL now cover every part except the LiPo and test pads.

Co-Authored-By: Claude Opus 5.5 (1M context) <noreply@anthropic.com>
Parts:
- removed U2: XIAO ESP32-S3, emg_wearable:XIAO_ESP32S3_SMD, symbol emg_wearable:XIAO_ESP32S3
- added C703, C704: 4.7uF, Capacitor_SMD:C_0603_1608Metric, symbol Device:C
- added C705, C708: 1uF, Capacitor_SMD:C_0603_1608Metric, symbol Device:C
- added C706: 10uF, Capacitor_SMD:C_0603_1608Metric, symbol Device:C
- added C707: 100nF, Capacitor_SMD:C_0603_1608Metric, symbol Device:C
- added J7: USB-C, Connector_USB:USB_C_Receptacle_HRO_TYPE-C-31-M-12, symbol Connector:USB_C_Receptacle_USB2.0_16P
- added R701, R702: 5.1k, Resistor_SMD:R_0603_1608Metric, symbol Device:R
- added R703, R704: 10k, Resistor_SMD:R_0603_1608Metric, symbol Device:R
- added TP10: BOOT (IO0), TestPoint:TestPoint_Pad_D1.0mm, symbol Connector:TestPoint
- added TP9: EN (reset), TestPoint:TestPoint_Pad_D1.0mm, symbol Connector:TestPoint
- added U2: ESP32-S3-MINI-1-N8, emg_wearable:ESP32-S3-MINI-1, symbol RF_Module:ESP32-S3-MINI-1
- added U7: USBLC6-2SC6, Package_TO_SOT_SMD:SOT-23-6, symbol Power_Protection:USBLC6-2SC6
- added U8: MCP73831T-2ACI/OT, Package_TO_SOT_SMD:SOT-23-5, symbol Battery_Management:MCP73831-2-OT
- added U9: AP2112K-3.3TRG1, Package_TO_SOT_SMD:SOT-23-5, symbol Regulator_Linear:AP2112K-3.3
- J3: footprint emg_wearable:LiPo_SolderPads_2x2.0x3.0mm_P3.5mm -> emg_wearable:LiPo_SolderPads_2x1.5x2.5mm_P2.6mm
Connections:
- net +3V3: now also C706.1, C707.1, R704.1, U2.3 (3V3), U9.5 (VOUT)
- net ADS_CS: now also U2.19 (IO15)
- net ADS_DRDY: now also U2.20 (IO16)
- net ADS_RESET: now also U2.22 (IO18)
- net ADS_START: now also U2.21 (IO17)
- net AGND: now also C703.2, C704.2, C705.2, C706.2, C707.2, C708.2, J7.A1 (GND), J7.A12 (GND), J7.B1 (GND), J7.B12 (GND), J7.SH (SHIELD), R701.2, R702.2, R703.2, U2.1 (GND), U2.2 (GND), U2.42 (GND), U2.43 (GND), U2.46 (GND), U2.47 (GND), U2.48 (GND), U2.49 (GND), U2.50 (GND), U2.51 (GND), U2.52 (GND), U2.53 (GND), U2.54 (GND), U2.55 (GND), U2.56 (GND), U2.57 (GND), U2.58 (GND), U2.59 (GND), U2.60 (GND), U2.61 (GND), U2.62 (GND), U2.63 (GND), U2.64 (GND), U2.65 (GND), U7.2 (GND), U8.2 (V_{SS}), U9.2 (GND)
- net SPI_MISO: now also U2.17 (IO13)
- net SPI_MOSI: now also U2.18 (IO14)
- net SPI_SCK: now also U2.16 (IO12)
- net VBAT: now also C704.1, U8.3 (V_{BAT})
- net VBUS: now also C703.1, J7.A4 (VBUS), J7.A9 (VBUS), J7.B4 (VBUS), J7.B9 (VBUS), U7.5 (VBUS), U8.4 (V_{DD})
- net VSYS: now also C705.1, U9.1 (VIN), U9.3 (EN)
- new net CHG_PROG: R703.1, U8.5 (PROG)
- new net ESP_BOOT: TP10.1, U2.4 (IO0)
- new net ESP_EN: C708.1, R704.2, TP9.1, U2.45 (EN)
- new net USB_CC1: J7.A5 (CC1), R701.1
- new net USB_CC2: J7.B5 (CC2), R702.1
- new net USB_DN: J7.A7 (D-), J7.B7 (D-), U2.23 (USB_D-), U7.3 (I/O2), U7.4 (I/O2)
- new net USB_DP: J7.A6 (D+), J7.B6 (D+), U2.24 (USB_D+), U7.1 (I/O1), U7.6 (I/O1)
- no-connect marks 14 -> 43
Other:
- note added: "LiPo: J3 = two solder pads for a protected LiPo. U8 MCP73831 charges it from USB at 100 mA (R_PROG 10k)."
- note added: "MCU: ESP32-S3-MINI-1-N8 (PCB antenna, keep copper out of the antenna end). Native USB on IO19/IO20 through USBLC6 ESD to USB-C. ADS1298 SPI: IO12 SCLK, IO13 DOUT (MISO), IO14 DIN (MOSI), IO15 CS, IO16 DRDY, IO17 START, IO18 RESET. Flashing over USB uses the built-in USB-Serial-JTAG. If it ever stops enumerating: short TP10 (IO0) to GND, then tap TP9 (EN) to GND. Charger U8 MCP73831 at 100 mA (R70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"
- note added: "POWER: USB-C 5V (D101) / LiPo (Q101) auto power path -> VSYS -> U6 LP5907 3.0 V -> +3V0_A (ADS1298 AVDD) and U9 AP2112K 3.3 V -> +3V3 (ESP32-S3, ADS1298 DVDD). U6 EN = +3V3, so the AFE is off whenever the MCU rail is off."
- note removed: "LiPo: J3 = two solder pads for the protected LiPo leads. XIAO BAT+/BAT- (U2 15/16) are under the module."
- note removed: "POWER: USB 5V (D101) / LiPo (Q101) auto power path -> VSYS -> U6 LP5907 3.0 V -> +3V0_A (ADS1298 AVDD) U6 EN = XIAO 3V3, so the AFE is off whenever the ESP32 is off. DVDD = XIAO 3V3."
